Commit message: teleop

File: urdf/virat.urdf (robot description, URDF)
Before this commit: robot virat, 4 links, 3 joints
Links:
- link bot2: mass 5 -> 100; geometry collision mesh filename=package://Gazebo_Virat/models/bot2/meshes/bot2.dae scale=0.25 0.25 0.25; visual mesh filename=package://Gazebo_Virat/models/bot2/meshes/bot2.dae scale=0.25 0.25 0.25
- link castors1: mass 0.1 -> 1; geometry collision mesh filename=package://Gazebo_Virat/models/castors1/meshes/castors1.dae scale=0.25 0.25 0.25; visual mesh filename=package://Gazebo_Virat/models/castors1/meshes/castors1.dae scale=0.25 0.25 0.25
- link left_wheel: mass 0.5 -> 5; geometry collision mesh filename=package://Gazebo_Virat/models/tyre1/meshes/tyre1.dae scale=0.25 0.25 0.25; visual mesh filename=package://Gazebo_Virat/models/tyre1/meshes/tyre1.dae scale=0.25 0.25 0.25
- link right_wheel: mass 0.5 -> 5; geometry collision mesh filename=package://Gazebo_Virat/models/tyre1/meshes/tyre1.dae scale=0.25 0.25 0.25; visual mesh filename=package://Gazebo_Virat/models/tyre1/meshes/tyre1.dae scale=0.25 0.25 0.25

Commit message: Added Camera

File: urdf/virat.urdf (robot description, URDF)
Before this commit: robot virat, 4 links, 3 joints
Links:
- added link camera_link, mass 1e-5; collision box size=0.05 0.05 0.05; visual box size=0.05 0.05 0.05
- link bot2: mass 100 -> 200
- link castors1: mass 1 -> 20
- link left_wheel: mass 5 -> 10
- link right_wheel: mass 5 -> 10
Joints:
- added joint camera_joint: type fixed, parent bot2, child camera_link, origin xyz=0.2 0 0.27 rpy=0 1 0, axis 0 1 0
- joint rwheel_bot2: axis 0 1 0 -> 0 0.3 0

Commit message: msg type created

File: urdf/virat.urdf (robot description, URDF)
Before this commit: robot virat, 5 links, 4 joints
Joints:
- joint camera_joint: origin xyz=0.2 0 0.27 rpy=0 1 0 -> xyz=0.2 0 0.27 rpy=0 0.5 0
